File: PCB/PCB_V1/PCB_V1.kicad_sch (KiCad schematic)
At the start: 7 parts, among them J1 Conn_01x02_Female, J2 Conn_01x04_Male, J3 Screw_Terminal_01x02, U1 NE555P

Commit message: YEEPPO
Connections:
- net Electrode_2 is gone; now on net Analog_Calib: C1.2, J1.1 (Pin_1), U1.2 (TR), U1.6 (THR)
- net Analog_Calib: no longer J1.2 (Pin_2), R3.2, U1.7 (DIS)
- new net Electrode_1: J1.2 (Pin_2), R3.2, U1.7 (DIS)
Changed lines of the file:
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@@
 (kicad_sch (version 20211123) (generator eeschema)
   (paper "A4")
-  (junction (at 142.24 46.99) (diameter 0) (color 0 0 0 0)
-  )
   (junction (at 82.55 71.12) (diameter 0) (color 0 0 0 0)
   )
@@
     (stroke (width 0) (type default) (color 0 0 0 0))
   )
-  (wire (pts (xy 142.24 46.99) (xy 152.4 46.99))
-    (stroke (width 0) (type default) (color 0 0 0 0))
-  )
   (wire (pts (xy 132.08 78.74) (xy 125.73 78.74))
     (stroke (width 0) (type default) (color 0 0 0 0))
@@
     (stroke (width 0) (type default) (color 0 0 0 0))
   )
-  (wire (pts (xy 142.24 46.99) (xy 142.24 54.61))
+  (wire (pts (xy 142.24 41.91) (xy 142.24 54.61))
     (stroke (width 0) (type default) (color 0 0 0 0))
   )
@@
   )
   (wire (pts (xy 64.77 49.53) (xy 64.77 31.75))
-    (stroke (width 0) (type default) (color 0 0 0 0))
-  )
-  (wire (pts (xy 142.24 41.91) (xy 142.24 46.99))
     (stroke (width 0) (type default) (color 0 0 0 0))
   )
@@
     )
   )
-  (global_label "Analog_Calib" (shape input) (at 152.4 46.99 0) (fields_autoplaced)
-    (effects (font (size 1.27 1.27)) (justify left))
-    (property "Intersheet References" "${INTERSHEET_REFS}" (id 0) (at 166.9688 46.9106 0)
-      (effects (font (size 1.27 1.27)) (justify left) hide)
+  (global_label "Analog_Calib" (shape input) (at 125.73 59.69 270) (fields_autoplaced)
+    (effects (font (size 1.27 1.27)) (justify right))
+    (property "Intersheet References" "${INTERSHEET_REFS}" (id 0) (at 125.8094 74.2588 90)
+      (effects (font (size 1.27 1.27)) (justify right) hide)
     )
   )
